File: IEEE-Macropad.kicad_pcb (KiCad board)
At the start: 2 copper layers, 98.4 x 76.2 mm, 48 parts, among them SW1 SW_Push, U1 ATmega32U4-A, Y1 16MHz

Commit message: fill zones
Routing:
- added copper zone on B.Cu, net GND
Other:
- board text added: "Gianna Wong IEEE Macropad"
Changed lines of the file:
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@@
 		(at 138.11875 26.45625 -90)
 		(property "Reference" "USB1"
-			(at 2.032 0 180)
+			(at 2.032 0.00625 180)
 			(layer "B.SilkS")
 			(effects
@@
 		(at 138.0375 96.575 180)
 		(property "Reference" "SW1"
-			(at 0 -4.064 180)
+			(at -6.425 -0.2625 180)
 			(layer "B.SilkS")
 			(effects
@@
 		(tags "resistor")
 		(property "Reference" "R3"
-			(at 0 1.65 90)
+			(at 3.29375 0 90)
 			(layer "B.SilkS")
 			(effects
@@
 		(tags "SOD-123")
 		(property "Reference" "D4"
-			(at 0 2 270)
+			(at -4.03125 0 270)
 			(layer "B.SilkS")
 			(effects
@@
 		)
 		(fp_text user "${REFERENCE}"
-			(at 0 2 270)
+			(at -4.03125 0 270)
 			(layer "B.Fab")
 			(effects
@@
 		(tags "resistor")
 		(property "Reference" "R1"
-			(at 0 1.65 90)
+			(at -3.175 0 90)
 			(layer "B.SilkS")
 			(effects
@@
 		(tags "SOD-123")
 		(property "Reference" "D16"
-			(at 0 2 270)
+			(at -4.03125 0 270)
 			(layer "B.SilkS")
 			(effects
@@
 		)
 		(fp_text user "${REFERENCE}"
-			(at 0 2 270)
+			(at -4.03125 0 270)
 			(layer "B.Fab")
 			(effects
@@
 		(tags "capacitor")
 		(property "Reference" "C5"
-			(at 0 1.68 270)
+			(at 3.01875 0 270)
 			(layer "B.SilkS")
 			(effects
@@
 		(tags "resistor")
 		(property "Reference" "R2"
-			(at 0 1.65 90)
+			(at 3.29375 0 90)
 			(layer "B.SilkS")
 			(effects
@@
 		(tags "SOD-123")
 		(property "Reference" "D12"
-			(at 0 2 270)
+			(at -3.90625 0 270)
 			(layer "B.SilkS")
 			(effects
@@
 		)
 		(fp_text user "${REFERENCE}"
-			(at 0 2 270)
+			(at -3.90625 0 270)
 			(layer "B.Fab")
 			(effects
@@
 		(tags "capacitor")
 		(property "Reference" "C2"
-			(at 0 1.68 270)
+			(at 0 -3.33125 270)
 			(layer "B.SilkS")
 			(effects
@@
 		(tags "SOD-123")
 		(property "Reference" "D8"
-			(at 0 2 270)
+			(at -4.03125 0 270)
 			(layer "B.SilkS")
 			(effects
@@
 		)
 		(fp_text user "${REFERENCE}"
-			(at 0 2 270)
+			(at -4.03125 0 270)
 			(layer "B.Fab")
 			(effects
@@
 		(tags "capacitor")
 		(property "Reference" "C1"
-			(at 0 1.68 90)
+			(at 0 -3.175 90)
 			(layer "B.SilkS")
 			(effects
@@
 		(layer "Edge.Cuts")
 	)
+	(gr_text "Gianna Wong\nIEEE Macropad"
+		(at 146.05 84.93125 0)
+		(layer "B.SilkS")
+		(effects
+			(font
+				(size 1 1)
+				(thickness 0.1)
+			)
+			(justify left bottom mirror)
+		)
+	)
 	(segment
 		(start 130.96875 46.0375)
@@
 	)
 	(segment
-		(start 139.71875 30.95625)
-		(end 139.71875 31.83125)
-		(width 0.381)
-		(layer "B.Cu")
-		(net 1)
-	)
-	(segment
 		(start 131.6375 64.95)
 		(end 132.7685 64.95)
@@
 	)
 	(segment
-		(start 139.71875 31.83125)
-		(end 140.49375 32.60625)
-		(width 0.381)
-		(layer "B.Cu")
-		(net 1)
-	)
-	(segment
 		(start 133.35 98.425)
 		(end 132.55625 97.63125)
@@
 	)
 	(segment
+		(start 140.49375 32.60625)
+		(end 139.71875 31.83125)
+		(width 0.381)
+		(layer "B.Cu")
+		(net 1)
+	)
+	(segment
+		(start 139.71875 31.83125)
+		(end 139.71875 30.95625)
+		(width 0.381)
+		(layer "B.Cu")
+		(net 1)
+	)
+	(segment
 		(start 130.1875 64.15)
 		(end 131.6375 64.15)
@@
 	)
 	(segment
-		(start 131.31675 66.07075)
-		(end 131.6375 65.75)
-		(width 0.254)
-		(layer "B.Cu")
-		(net 37)
-	)
-	(segment
 		(start 127.79375 46.099394)
 		(end 127.79375 65.204178)
@@
 	)
 	(segment
-		(start 128.660322 66.07075)
-		(end 131.31675 66.07075)
+		(start 130.6335 65.75)
+		(end 131.6375 65.75)
 		(width 0.254)
 		(layer "B.Cu")
@@
 	)
 	(segment
+		(start 128.660322 66.07075)
+		(end 130.31275 66.07075)
+		(width 0.254)
+		(layer "B.Cu")
+		(net 37)
+	)
+	(segment
+		(start 130.31275 66.07075)
+		(end 130.6335 65.75)
+		(width 0.254)
+		(layer "B.Cu")
+		(net 37)
+	)
+	(segment
 		(start 137.31875 33.89375)
 		(end 136.525 34.6875)
@@
 		(net 39)
 	)
+	(zone
+		(net 1)
+		(net_name "GND")
+		(layer "B.Cu")
+		(hatch edge 0.5)
+		(priority 1)
+		(connect_pads
+			(clearance 0.5)
+		)
+		(min_thickness 0.25)
+		(filled_areas_thickness no)
+		(fill yes
+			(thermal_gap 0.5)
+			(thermal_bridge_width 0.5)
+		)
+		(polygon
+			(pts
+				(xy 143.66875 42.06875) (xy 143.66875 57.94375) (xy 130.96875 57.94375) (xy 130.96875 42.06875)
+			)
+		)
+	)
+	(zone
+		(net 1)
+		(net_name "GND")
+		(layer "B.Cu")
+		(hatch edge 0.5)
+		(priority 2)
+		(connect_pads
+			(clearance 0.5)
+		)
+		(min_thickness 0.25)
+		(filled_areas_thickness no)
+		(fill yes
+			(thermal_gap 0.5)
+			(thermal_bridge_width 0.5)
+		)
+		(polygon
+			(pts
+				(xy 132.55625 59.53125) (xy 132.55625 69.05625) (xy 142.08125 69.05625) (xy 142.08125 59.53125)
+			)
+		)
+	)
+	(zone
+		(net 1)
+		(net_name "GND")
+		(layer "B.Cu")
+		(hatch edge 0.5)
+		(connect_pads
+			(clearance 0.5)
+		)
+		(min_thickness 0.25)
+		(filled_areas_thickness no)
+		(fill yes
+			(thermal_gap 0.5)
+			(thermal_bridge_width 0.5)
+		)
+		(polygon
+			(pts
+				(xy 134.9375 24.60625) (xy 134.9375 31.75) (xy 141.2875 31.75) (xy 141.2875 24.60625)
+			)
+		)
+	)
 )
